File: icarus_interface.sch (KiCad schematic (older format))
At the start: 48 parts, among them IC1 MC74VHC1GT50DBVT1G, IC2 TPS54540BDDA, J1 MEZZANINE, J2 MEZZANINE, J3 4pin_header, J4 4pin_header, J5 4pin_header

Commit message: update
Connections:
- net +3V3: no longer S2.19 (3V3), S2.2 (3V3)
- net HB_RX1: now also J5.1, S2.15 (RX); no longer J5.2
- net HB_TX1: now also J5.2; no longer J5.1
- net RPI_SCL1: no longer names the net of J1.56
- net RPI_SDA1: no longer names the net of J1.58
- no-connect marks 136 -> 140
Other:
- note added: "GPIO09"
- note added: "GPIO10"
- note added: "GPIO11"
- note added: "GPIO14"
- note added: "GPIO15"
- note added: "GPIO17"
- note added: "GPIO18"
- note added: "GPIO22"
- note added: "GPIO23"
- note added: "GPIO24"
- note added: "GPIO25"
- note added: "GPIO27"
Changed lines of the file:
@@
 	1    0    0    -1
 $EndComp
-$Comp
-L power:+3.3V #PWR08
-U 1 1 6047C834
-P 3600 6900
-F 0 "#PWR08" H 3600 6750 50  0001 C CNN
-F 1 "+3.3V" H 3615 7073 50  0000 C CNN
-F 2 "" H 3600 6900 50  0001 C CNN
-F 3 "" H 3600 6900 50  0001 C CNN
-	1    3600 6900
-	1    0    0    -1
-$EndComp
-Wire Wire Line
-	3800 6950 3600 6950
-Wire Wire Line
-	3600 6950 3600 6900
-Wire Wire Line
-	3800 7050 3600 7050
-Wire Wire Line
-	3600 7050 3600 6950
-Connection ~ 3600 6950
 Wire Wire Line
 	1450 6950 1250 6950
@@
 HB_TX1
 Text Label 10200 3750 2    50   ~ 0
-HB_RX1
+HB_TX1
 Text Label 4900 7150 0    50   ~ 0
 LED_4_n
@@
 Text Label 2800 3000 0    50   ~ 0
 RPI_MOSI0
-Text Label 2800 3600 0    50   ~ 0
-RPI_SCL1
-Text Label 2800 3700 0    50   ~ 0
-RPI_SDA1
 Text Label 2800 3300 0    50   ~ 0
 LED_2_n
@@
 Text Label 2800 5400 0    50   ~ 0
 RPI_RUN_PG
-Wire Wire Line
-	2800 3700 2500 3700
-Wire Wire Line
-	2800 3600 2500 3600
 Wire Wire Line
 	2800 3300 2500 3300
@@
 $EndComp
 Text Label 10200 3650 2    50   ~ 0
-HB_TX1
+HB_RX1
 Text Label 2550 6550 0    50   ~ 0
 HB_TX6
@@
 Connection ~ 2800 4700
 $Comp
-L power:+3.3VA #PWR?
+L power:+3.3VA #PWR0104
 U 1 1 60E9B786
 P 7200 900
-F 0 "#PWR?" H 7200 750 50  0001 C CNN
+F 0 "#PWR0104" H 7200 750 50  0001 C CNN
 F 1 "+3.3VA" H 7215 1073 50  0000 C CNN
 F 2 "" H 7200 900 50  0001 C CNN
@@
 $EndComp
 $Comp
-L power:+3.3VA #PWR?
+L power:+3.3VA #PWR0105
 U 1 1 60E9CCF3
 P 7550 900
-F 0 "#PWR?" H 7550 750 50  0001 C CNN
+F 0 "#PWR0105" H 7550 750 50  0001 C CNN
 F 1 "+3.3VA" H 7565 1073 50  0000 C CNN
 F 2 "" H 7550 900 50  0001 C CNN
@@
 $EndComp
 $Comp
-L power:+3.3VA #PWR?
+L power:+3.3VA #PWR0106
 U 1 1 60E9CE72
 P 8050 900
-F 0 "#PWR?" H 8050 750 50  0001 C CNN
+F 0 "#PWR0106" H 8050 750 50  0001 C CNN
 F 1 "+3.3VA" H 8065 1073 50  0000 C CNN
 F 2 "" H 8050 900 50  0001 C CNN
@@
 	1    0    0    -1
 $EndComp
+Text Notes 550  2900 0    50   ~ 0
+GPIO25
+Text Notes 550  3100 0    50   ~ 0
+GPIO24
+Text Notes 550  3200 0    50   ~ 0
+GPIO23
+Text Notes 550  3300 0    50   ~ 0
+GPIO18
+Text Notes 550  3400 0    50   ~ 0
+GPIO15
+Text Notes 550  3600 0    50   ~ 0
+GPIO14
+Text Notes 3250 2700 0    50   ~ 0
+GPIO11
+Text Notes 3250 2800 0    50   ~ 0
+GPIO09
+Text Notes 3250 3000 0    50   ~ 0
+GPIO10
+Text Notes 3250 3100 0    50   ~ 0
+GPIO22
+Text Notes 3250 3200 0    50   ~ 0
+GPIO27
+Text Notes 3250 3300 0    50   ~ 0
+GPIO17
+NoConn ~ 2500 3600
+NoConn ~ 2500 3700
+NoConn ~ 3800 6950
+NoConn ~ 3800 7050
+Text Label 4900 6650 0    50   ~ 0
+HB_RX1
 $EndSCHEMATC

Commit message: update
Connections:
- net +3.3VA: now also J1.86
- no-connect marks 140 -> 139
Changed lines of the file:
@@
 Title "ICARUS_INTERFACE"
 Date "2021-02-22"
-Rev "0.3"
+Rev "1.0"
 Comp "EPFL ROCKETTEAM"
 Comment1 "Iacopo Sprenger"
@@
 NoConn ~ 2500 5300
 NoConn ~ 2500 5200
-NoConn ~ 2500 5100
 NoConn ~ 1500 4600
 NoConn ~ 1500 4500
@@
 NoConn ~ 3750 1700
 NoConn ~ 3750 1600
-NoConn ~ 3750 1400
 NoConn ~ 3750 1300
 Wire Wire Line
@@
 Text Label 4900 6650 0    50   ~ 0
 HB_RX1
+Wire Wire Line
+	2500 5100 2800 5100
+Wire Wire Line
+	2800 5100 2800 5000
+Connection ~ 2800 5000
+NoConn ~ 3750 1400
 $EndSCHEMATC

Commit message: quick modifs
Parts:
- added C12: 100u, Capacitor_Tantalum_SMD:CP_EIA-3528-21_Kemet-B, symbol Device:CP
- R12: value 511k -> 147k
- R13: value 82.5k -> 32.4k
Connections:
- net +5V: now also C12.1
- net GND: now also C12.2
Changed lines of the file:
@@
 Connection ~ 1350 4400
 Wire Wire Line
-	1350 4400 1350 5950
+	1350 4400 1350 5350
 Wire Wire Line
 	1500 4700 1200 4700
@@
 P 6700 5300
 F 0 "R12" H 6770 5346 50  0000 L CNN
-F 1 "511k" H 6770 5255 50  0000 L CNN
+F 1 "147k" H 6770 5255 50  0000 L CNN
 F 2 "Resistor_SMD:R_0805_2012Metric" V 6630 5300 50  0001 C CNN
 F 3 "~" H 6700 5300 50  0001 C CNN
@@
 P 6700 5800
 F 0 "R13" H 6770 5846 50  0000 L CNN
-F 1 "82.5k" H 6770 5755 50  0000 L CNN
+F 1 "32.4k" H 6770 5755 50  0000 L CNN
 F 2 "Resistor_SMD:R_0805_2012Metric" V 6630 5800 50  0001 C CNN
 F 3 "~" H 6700 5800 50  0001 C CNN
@@
 Connection ~ 2800 5000
 NoConn ~ 3750 1400
+$Comp
+L Device:CP C12
+U 1 1 606FA6B8
+P 800 4900
+F 0 "C12" H 918 4946 50  0000 L CNN
+F 1 "100u" H 918 4855 50  0000 L CNN
+F 2 "Capacitor_Tantalum_SMD:CP_EIA-3528-21_Kemet-B" H 838 4750 50  0001 C CNN
+F 3 "~" H 800 4900 50  0001 C CNN
+	1    800  4900
+	1    0    0    -1
+$EndComp
+Wire Wire Line
+	800  4700 800  4750
+Connection ~ 800  4700
+Wire Wire Line
+	800  5050 800  5350
+Wire Wire Line
+	800  5350 1350 5350
+Connection ~ 1350 5350
+Wire Wire Line
+	1350 5350 1350 5950
 $EndSCHEMATC
