File: icarus_interface.kicad_pcb (KiCad board)
At the start: 2 copper layers, 70.5 x 42.5 mm, 52 parts, among them IC1 MC74VHC1GT50DBVT1G, IC2 TPS54540BDDA, J1 MEZZANINE, J2 MEZZANINE, J3 4pin_header, J4 4pin_header, J5 4pin_header

Commit message: tst
Routing:
- net GND: track 5.09 -> 92.4 mm
- net /RPI_GP4: track 51.8 -> 52.4 mm

Commit message: update
Parts:
- D1, D2, D8, IC1, R11, R19, R2, R3: moved to F.Cu
- moved G*** 17.2 mm to (110.5, 65.3)
Connections:
- net /RPI_SCL1 renamed Net-(J1-Pad56)
- net /RPI_SDA1 renamed Net-(J1-Pad58)
- J5 pad 1: /HB_TX1 -> /HB_RX1
- J5 pad 2: /HB_RX1 -> /HB_TX1
- S2 pad 15: Net-(S2-Pad15) -> /HB_RX1
- S2 pad 19: +3V3 -> Net-(S2-Pad19)
- S2 pad 2: +3V3 -> Net-(S2-Pad2)
Routing:
- net GND: track 92.4 -> 111.1 mm, vias 14 -> 20
- net +5V: track 57.6 -> 48.7 mm, vias 11 -> 17
- net +3.3VA: track 44.7 -> 51.4 mm, vias 3 -> 2
- net /HB_RX1: track 0.00 -> 6.15 mm
- net /HB_RX: track 6.15 -> 0.00 mm
- net /HB_TX1: track 0.00 -> 6.15 mm
- net /HB_TX: track 6.15 -> 0.00 mm
- net /RPI_GP1: track 59.9 -> 57.5 mm
- net /LED_ACT_n: track 17.3 -> 19.7 mm, vias 1 -> 0
- net /RPI_GP3: track 54.8 -> 52.6 mm
- net Net-(IC2-Pad5): track 1.37 -> 3.37 mm
- net /HB_PWM1: track 42.9 -> 44.7 mm
- net /RPI_GP4: track 52.4 -> 50.6 mm
- net /LED_PWR_n: track 28.4 -> 26.7 mm, vias 1 -> 2
- net /HB_PWM2: track 43.8 -> 45.2 mm
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Other:
- board text added: "RX"
- board text added: "TX"

Commit message: update
Connections:
- J1 pad 86: Net-(J1-Pad86) -> +3.3VA
Routing:
- net +3.3VA: track 51.4 -> 55.2 mm

Commit message: quick modifs
Parts:
- removed the C10 at (139.2, 39.1)
- added C12: 100u, Capacitor_Tantalum_SMD:CP_EIA-3528-21_Kemet-B, B.Cu at (139.2, 39.9)
- IC1: footprint pegasus_interface:SOT65P210X110-5N -> icarus_interface:SOT65P210X110-5N
- J1, J2: footprint pegasus_interface:DF40HC30100DS04V51 -> icarus_interface:MEZZANINE

Commit message: sync
Parts:
- added REF**: MountingHole_2.7mm_M2.5_ISO7380, icarus_interface:CM4_Mounting_hole, F.Cu at (91.1, 67.1)
- added REF**: MountingHole_2.7mm_M2.5_ISO7380, icarus_interface:CM4_Mounting_hole, F.Cu at (139.1, 67.1)
- added REF**: MountingHole_2.7mm_M2.5_ISO7380, icarus_interface:CM4_Mounting_hole, F.Cu at (139.1, 34.1)
- added REF**: MountingHole_2.7mm_M2.5_ISO7380, icarus_interface:CM4_Mounting_hole, F.Cu at (91.1, 34.1)
Routing:
- net GND: vias 20 -> 32
- net +3.3VA: vias 2 -> 3
- net (no net): vias 4 -> 0
